File: PCB/telescope_board.kicad_pcb (KiCad board)
At the start: 2 copper layers, 80 x 100 mm, 39 parts

Commit message: final
Parts:
- C1: renamed from 100µF 12V
- C2: renamed from 220µF 5V BULK
- C5, C6: renamed from 100µF VMOT
- C7, C8: renamed from 100nF 
- C9: renamed from 100nF 5V
- D1: renamed from 6.8V ZENER
- F1: renamed from FUSE 4A; footprint Fuse:Fuse_1812_4532Metric -> Fuse:Fuse_2920_7451Metric
- F2: renamed from FUSE 1.5A PI
- J1: renamed from 12V DC IN
- JP1: renamed from MS1 (ALT)
- JP2: renamed from MS2 (ALT)
- JP3: renamed from MS1 (AZ)
- JP4: renamed from MS2 (AZ)
- J_GPS1: renamed from GPS MODULE
- J_LIM1: renamed from LIMIT ALT
- J_LIM2: renamed from LIMIT AZ
- J_MOT1: renamed from MOTOR ALTITUDE
- J_MOT2: renamed from MOTOR AZIMUTH
- J_MP1584: renamed from MP1584 BUCK
- J_PI1: renamed from RASPBERRY PI ZERO
- J_TMC1: renamed from TMC2209 ALTITUDE
- J_TMC2: renamed from TMC2209 AZIMUTH
- Q1: renamed from REVERSE PROTECT
- R1: renamed from 10k R
- R2: renamed from 10k 
- moved F1 2.06 mm to (181.7, 45.1)
- renumbered 100nF to C10, 100nF to C11, 22µF to C3, 100nF to C4, 10k to R3, +12V to TP1, +5V to TP2, +3V3 to TP3, GND to TP4, STEP1 to TP5, GPS_RX to TP6, AMS1117 to U1
Routing:
- net Net-(D1-A): track 7.11 -> 8.87 mm
- net Net-(F1-Pad1): track 7.25 -> 8.82 mm
