File: PCB/telescope_board.kicad_sch (KiCad schematic)
At the start: 39 parts, among them J1 Barrel_Jack_Switch, Q1 AO3401A, U1 AMS1117-3.3

Commit message: final
Parts:
- F1: footprint Fuse:Fuse_1812_4532Metric -> Fuse:Fuse_2920_7451Metric
Changed lines of the file:
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@@
 			)
 		)
-		(property "Footprint" "Fuse:Fuse_1812_4532Metric"
+		(property "Footprint" "Fuse:Fuse_2920_7451Metric"
 			(at 92.71 85.09 0)
 			(effects
